Commit message: updated urdf model and trig calcs

File: mercerbot_description/urdf/mercerbot.urdf.xacro (robot description, xacro)
@@ -5,4 +5,6 @@
     <xacro:property name="effort" value="30.0" />
     <xacro:property name="velocity" value="10.0" />
+  <!-- Include ros2_control Plugins -->
+    <xacro:include filename="$(find arduinobot_description)/urdf/arduinobot_ros2_control.xacro" />
   <!-- Include Color Parameters -->
   <xacro:include filename="$(find mercerbot_description)/urdf/xkcd_colors.urdf.xacro" />
@@ -60,9 +62,9 @@
   <link name="elbow_link_actual">
     <visual>
-      <origin xyz=".05 0 0.04" rpy="0 0 0"/>
+      <origin xyz="0.02 0 0.02" rpy="0 0 0"/>
       <geometry>
-        <box size="0.01 0.02 0.08"/>
+        <box size="0.01 0.01 0.04"/>
       </geometry>
-      <material name="pink"/>
+      <material name="green"/>
     </visual>
   </link>
@@ -121,13 +123,13 @@
         <parent link="shoulder_link"/>
         <child link = "elbow_link_corrected"/>
-        <origin xyz="0 0 0.08" rpy="${PI/2} 0 0"/>
+        <origin xyz="0 0 0.08" rpy="-${PI/2} 0 0"/>
         <axis xyz="1 0 0"/>
         <limit lower="-${PI / 2}" upper="${PI / 2}"
                effort="${effort}" velocity="${velocity}"/>
     </joint>
-<joint name ="joint_3_actual" type="revolute">
-        <parent link="shoulder_link"/>
+    <joint name ="joint_3" type="revolute">
+        <parent link="base_plate"/>
         <child link = "elbow_link_actual"/>
-        <origin xyz="0 0 0.08" rpy="${PI/2} 0 0"/>
+        <origin xyz="0 0 0.02" rpy="${PI/2} 0 0"/>
         <axis xyz="1 0 0"/>
         <limit lower="-${PI / 2}" upper="${PI / 2}"

Commit message: updated msg

File: mercerbot_description/urdf/mercerbot.urdf.xacro (robot description, xacro)
@@ -71,7 +71,7 @@
    <link name="claw_support">
       <visual>
-          <origin rpy="0 1.57 0" xyz="0 0 0"/>
+          <origin rpy="0 0 0" xyz="0 0 0"/>
           <geometry>
-              <box size="0.01 0.02 0.03"/>
+              <box size="0.01 0.02 0.01"/>
           </geometry>
         <material name="white"/>
@@ -80,7 +80,7 @@
     <link name="gripper_right">
           <visual>
-              <origin rpy="0 0 0" xyz="0 0 0"/>
+              <origin rpy="${PI/2} 0 0" xyz="0 0 0"/>
               <geometry>
-                  <box size="0.005 0.005 0.03"/>
+                  <box size="0.005 0.005 0.015"/>
               </geometry>
               <material name="red"/>
@@ -89,7 +89,7 @@
       <link name="gripper_left">
           <visual>
-              <origin rpy="0 0 0" xyz="0 0 0"/>
+              <origin rpy="${PI/2} 0 0" xyz="0 0 0"/>
               <geometry>
-                  <box size="0.005 0.005 0.03"/>
+                  <box size="0.005 0.005 0.015"/>
               </geometry>
               <material name="green"/>
@@ -139,5 +139,5 @@
         <parent link="elbow_link_corrected"/>
         <child link = "claw_support"/>
-        <origin xyz="0 0.0 0.08"/>
+        <origin xyz="0 0.01 0.09" rpy="${PI} 0 0"/>
         <axis xyz="1 0 0"/>
         <limit lower="-${PI / 2}" upper="${PI / 2}"
@@ -147,5 +147,5 @@
           <parent link="claw_support"/>
           <child link = "gripper_right"/>
-          <origin xyz="-0.0125 -0.005 0.02"/>
+          <origin xyz="-0.005 -0.01 0.005" rpy="0 0 0"/>
           <axis xyz="0 0 1"/>
           <limit lower="-${PI / 2}" upper="0.0"
@@ -155,8 +155,9 @@
           <parent link="claw_support"/>
           <child link = "gripper_left"/>
-          <origin xyz="0.0125 -0.005 0.02"/>
+          <origin xyz="0.005 -0.01 0.005" rpy="0 0 0"/>
           <axis xyz="0 0 1"/>
-          <limit lower="-${PI / 2}" upper="0.0"
+          <limit lower="0.0" upper="${PI / 2}"
                 effort="${effort}" velocity="${velocity}"/>
+          <mimic joint="joint_4" multiplier="-1.0" offset="0.0"/>
       </joint>
 </robot>
